File: kicad/j_link_interface.kicad_sch (KiCad schematic)
At the start: 9 parts, among them J1 Conn_01x05_Pin, J2 SSW-110-02-G-D-RA-N, J3 FTSH-107-01-X-DV-K

Commit message: Updated with originally intended 0603 package for resistors. Changed the switch. Changed the IDC connector to a better matching one. Added release workflow.
Parts:
- removed H1, H2: MountingHole, local_library:MountingHole_2.2mm_M2, symbol Mechanical:MountingHole
- J1: Supplier (none) -> Digi-Key; SupplierPN (none) -> 1849-PR20206VBNN-ND
- J2: value SSW-110-02-G-D-RA-N -> SFH11-PBPC-D10-RA-BK; footprint local_library:SAMTEC_SSW-110-02-G-D-RA-N -> local_library:SFH11-PBPC-D10-RA-BK; LCSC C6236423 -> C3319874; MF Samtec -> Sullins Connector Solutions; MP SSW-110-02-G-D-RA-N -> SFH11-PBPC-D10-RA-BK; Supplier (none) -> Digi-Key; SupplierPN (none) -> S9205-ND
- J3: Supplier (none) -> Digi-Key; SupplierPN (none) -> SAM9449-ND
- R1: footprint Resistor_SMD:R_0201_0603Metric -> Resistor_SMD:R_0603_1608Metric; Supplier (none) -> Digi-Key; SupplierPN (none) -> 541-100HCT-ND
- R2, R3: footprint Resistor_SMD:R_0201_0603Metric -> Resistor_SMD:R_0603_1608Metric; Supplier (none) -> Digi-Key; SupplierPN (none) -> 541-1.00KHCT-ND
- S1: value EVQP7C01P -> (none); footprint local_library:SW_EVQ-P7C01P -> local_library:EVQP4HB3B; symbol PCM_JLCPCB-Connectors_Buttons:Tactile Button, 160gf, 12V, 50mA, 5.1mm -> local_library:EVQP42B3M; Height (none) -> 3.7; LCSC C388883 -> C485511; MP EVQP7C01P -> EVQP42B3M; Manufacturer_Name (none) -> Panasonic; Manufacturer_Part_Number (none) -> EVQP42B3M; Supplier (none) -> Digi-Key; SupplierPN (none) -> EVQ-P42B3MD
Connections:
- net GND: now also S1.2 (COM)
Other:
- moved on the sheet: R1
